File: drone_remote.kicad_sch (KiCad schematic)
At the start: 100 parts, among them J1 USBC, J10 HEADER_C, J2 BAT, J3 UART, J4 SWI, J5 OLDED_SMALL, J6 OLED_BIG, J7 RFM_SOCKET, J8 RFM_SOCKET, J9 HEADER_AB, Q1 PMOS, SW1 RST_BTN, SW2 PUSH_BTN_U, SW3 PUSH_BTN_L, SW4 PUSH_BTN_R, SW5 PUSH_BTN_D, SW6 ENC1, SW7 ENC2, SW8 SW_SPDT, U1 STM32F411RETx, U2 TC1262-33, U3 SN74ALVC14PWR, U4 SN74ALVC14PWR, U5 INA180A2, U6 FT230XS, X1 32.768KHZ, X2 8MHZ

Commit message: changes
Parts:
- removed J4: SWI, Connector_PinSocket_1.00mm:PinSocket_1x05_P1.00mm_Vertical, symbol Connector_Generic:Conn_01x05
- removed JP3: BLK_ON, Connector_PinSocket_1.27mm:PinSocket_1x02_P1.27mm_Vertical, symbol Jumper:Jumper_2_Open
- added J4: Conn_01x05_Pin, symbol Connector:Conn_01x05_Pin
- added JP1: Jumper_2_Bridged, symbol Jumper:Jumper_2_Bridged
- added R2: 5k, Resistor_SMD:R_0805_2012Metric, symbol Device:R_Small
- added R27: 47, Resistor_SMD:R_0805_2012Metric, symbol Device:R_Small
- L2: value L_UART -> 120R
Connections:
- net 3.3V is gone; now on net +3.3V: C16.1, C17.1, J5.1 (Pin_1), J6.2 (Pin_2), J7.1 (Pin_1), R16.2, R17.2, R18.1, R19.2, R20.2, R21.1, R22.1, R23.2, R24.2, R25.2, R26.2, U2.3 (VO), U3.14 (VCC), U4.14 (VCC), U5.5 (V+)
- net +3.3V: now also J4.1 (Pin_1), JP1.2 (B)
- net ADC_CURRENT_SENSE: no longer U5.1
- net GND: now also SW7.C, J4.5 (Pin_5), R2.2, R27.2; no longer J1.SH1 (SHIELD), J1.SH2 (SHIELD__1), J1.SH3 (SHIELD__2), J1.SH4 (SHIELD__3), J3.6 (Shield)
- net RFM__G0: no longer J7.9 (Pin_9)
- net RFM_nRST: no longer J7.8 (Pin_8)
- net SPI1_MOSI: no longer J7.6 (Pin_6)
- net SPI1_SCK: no longer J7.4 (Pin_4)
- net SPI2_NSS: no longer J6.7 (Pin_7)
- net ST7735_nRESET: no longer J6.5 (Pin_5)
- net SWCLK: now also J4.4 (Pin_4)
- net SWDIO: now also J4.2 (Pin_2)
- net USB_OTG_FS_DM: no longer D1.1 (A1), J1.A7 (DN1), U1.45 (PA12)
- net USB_OTG_FS_DP: no longer D2.1 (A1), J1.A6 (DP1), U1.44 (PA11)
- net at C32.2, SW1.1, SW1.3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: now also J4.3 (Pin_3)
- net VBUS: now reaches C14.2, D3.1 (A1), F1.1, J1.A4_B9 (VBUS)
- net VBUS: now also C18.2, J3.1 (VBUS), L2.1
- net +5V: now reaches J2.2 (Pin_2), Q1.3 (S)
- net at J6.8 (Pin_8), JP2.2 (B): now also JP1.1 (A)
- new net: J1.SH1 (SHIELD), J1.SH2 (SHIELD__1), J1.SH3 (SHIELD__2), J1.SH4 (SHIELD__3), R2.1
- new net: J3.6 (Shield), R27.1
- new net ADC_CURRENT: U5.1
- new net RFM_G0: J7.9 (Pin_9)
- new net RMF_nRST: J7.8 (Pin_8)
- new net SPI1-SCK: J7.4 (Pin_4)
- new net SPI1_MOSO: J7.6 (Pin_6)
- new net SPI2_nCS: J6.7 (Pin_7)
- new net ST77735_nRST: J6.5 (Pin_5)
- new net USB_OTG_FS_DM-: D1.1 (A1), J1.A7 (DN1), U1.44 (PA11)
- new net USB_OTG_FS_DP+: D2.1 (A1), J1.A6 (DP1), U1.45 (PA12)
Other:
- moved on the sheet: C18, J10, L2

Commit message: update
Parts:
- removed C10, C11: 12p, Capacitor_SMD:C_0402_1005Metric, symbol Device:C_Small
- removed C17: 0.1u, Capacitor_SMD:C_0805_2012Metric, symbol Device:C_Small
- removed D7: UART_TX, LED_SMD:LED_0201_0603Metric, symbol Device:LED
- removed D8: HEARTBEAT, Inductor_SMD:L_0201_0603Metric, symbol Device:LED
- removed J10: HEADER_C, Connector_PinSocket_1.27mm:PinSocket_2x16_P1.27mm_Vertical, symbol Connector_Generic:Conn_02x16_Counter_Clockwise
- removed J2: BAT, Connector_PinSocket_2.54mm:PinSocket_1x02_P2.54mm_Vertical, symbol Connector_Generic:Conn_01x02
- removed J5: OLDED_SMALL, Connector_PinSocket_1.00mm:PinSocket_1x04_P1.00mm_Vertical, symbol Connector_Generic:Conn_01x04
- removed J6: OLED_BIG, Connector_PinSocket_1.00mm:PinSocket_1x08_P1.00mm_Vertical, symbol Connector_Generic:Conn_01x08
- removed J7, J8: RFM_SOCKET, Connector_PinSocket_1.00mm:PinSocket_1x09_P1.00mm_Vertical, symbol Connector_Generic:Conn_01x09
- removed J9: HEADER_AB, Connector_PinSocket_1.27mm:PinSocket_2x16_P1.27mm_Vertical, symbol Connector_Generic:Conn_02x16_Counter_Clockwise
- removed JP2: BLK_OFF, Connector_PinSocket_1.27mm:PinSocket_1x02_P1.27mm_Vertical, symbol Jumper:Jumper_2_Open
- removed R14, R15: 660, Resistor_SMD:R_0805_2012Metric, symbol Device:R_Small
- removed R27: 47, Resistor_SMD:R_0805_2012Metric, symbol Device:R_Small
- removed R9: 0.1, Resistor_SMD:R_0805_2012Metric, symbol Device:R_Small
- removed SW2: PUSH_BTN_U, SW4_1825910-B_TEC:SW4_1825910-B_TEC, symbol SW4_1825910-B_TEC:1825910-6
- removed SW3: PUSH_BTN_L, SW4_1825910-B_TEC:SW4_1825910-B_TEC, symbol SW4_1825910-B_TEC:1825910-6
- removed SW4: PUSH_BTN_R, SW4_1825910-B_TEC:SW4_1825910-B_TEC, symbol SW4_1825910-B_TEC:1825910-6
- removed SW5: PUSH_BTN_D, SW4_1825910-B_TEC:SW4_1825910-B_TEC, symbol SW4_1825910-B_TEC:1825910-6
- removed SW8: SW_SPDT, symbol Switch:SW_SPDT
- removed U5: INA180A2, Package_TO_SOT_SMD:SOT-23-5, symbol Amplifier_Current:INA180A2
- removed X2: 8MHZ, CRYSTAL_ECS-80-18-5PX-TR_ECS:CRYSTAL_ECS-80-18-5PX-TR_ECS, symbol CRYSTAL_ECS-80-18-5PX-TR_ECS:ECS-80-18-5PX-TR
- added H1, H2, H3, H4: MountingHole, MountingHole:MountingHole_2.2mm_M2, symbol Mechanical:MountingHole
- added J2: Conn_01x02_Socket, Connector_PinHeader_2.54mm:PinHeader_1x02_P2.54mm_Vertical, symbol Connector:Conn_01x02_Socket
- added J5: Conn_01x04_Socket, Connector_PinSocket_2.54mm:PinSocket_1x04_P2.54mm_Vertical, symbol Connector:Conn_01x04_Socket
- added J6: Conn_01x08_Socket, Connector_PinSocket_2.54mm:PinSocket_1x08_P2.54mm_Vertical, symbol Connector:Conn_01x08_Socket
- added J7, J8: Conn_01x09_Socket, Connector_PinSocket_2.54mm:PinSocket_1x09_P2.54mm_Vertical, symbol Connector:Conn_01x09_Socket
- added JP4: Jumper_2_Bridged, Connector_PinHeader_2.54mm:PinHeader_1x02_P2.54mm_Vertical, symbol Jumper:Jumper_2_Bridged
- added SW2, SW3, SW4, SW5: RST_BTN, SW4_1825910-B_TEC:SW4_1825910-B_TEC, symbol Switch:SW_Push_Dual
- C10: renamed from C33; footprint Capacitor_SMD:C_0805_2012Metric -> Capacitor_SMD:C_0402_1005Metric
- C13: renamed from C12; value 36p -> 10p
- C14: renamed from C13; value 36p -> 10p
- C2, C3, C4, C5, C6, C7, C8, C9: footprint Capacitor_SMD:C_0805_2012Metric -> Capacitor_SMD:C_0402_1005Metric
- D1, D2, D3: footprint Diode_SMD:D_0201_0603Metric -> Diode_SMD:D_0402_1005Metric
- D6: value UART_RX -> HEARTBEAT; footprint LED_SMD:LED_0201_0603Metric -> Inductor_SMD:L_0201_0603Metric
- J1: footprint SAMESKY_UJ20-C-H-G-MSMT-3-P16-TR:SAMESKY_UJ20-C-H-G-MSMT-3-P16-TR -> drone_remote:GCT_USB4105-GF-A
- J4: footprint (none) -> Connector_PinHeader_2.54mm:PinHeader_1x05_P2.54mm_Vertical
- JP1: footprint (none) -> Connector_PinHeader_2.54mm:PinHeader_1x02_P2.54mm_Vertical
- L1, L2: footprint Inductor_SMD:L_0805_2012Metric -> Inductor_SMD:L_0603_1608Metric
- R2: value 5k -> 660
- R5: value 660 -> 10k
- X1: value 32.768KHZ -> 8MHZ; footprint (none) -> ECS-80-10:SMD_ECS-80-10-3M-TR_ECS
- renumbered C14 to C15, C15 to C16, C16 to C17, C18 to C19, C19 to C20, C20 to C21, C21 to C22, C22 to C23, C23 to C24, C24 to C26, C26 to C27, C27 to C28, C28 to C29, C29 to C30, C30 to C31, C31 to C32, C32 to C33
Connections:
- net PA10 is gone; now on net USART_RX: U1.43 (PA10)
- net PA9 is gone; now on net USART_TX: U1.42 (PA9)
- net PB8 is gone; now on net I2C1_SCL: U1.61 (PB8)
- net PB9 is gone; now on net I2C1_SDA: U1.62 (PB9)
- net ST7735_nRESET is gone; now on net ENC1_BTN: U1.17 (PA3)
- net +3.3V: now also J5.4 (Pin_4), J6.2 (Pin_2), J7.1 (Pin_1), JP4.1 (A)
- net +5V: now also J2.2 (Pin_2)
- net ADC_VOLTAGE: now also U1.27 (PB1); no longer U1.9 (PC1)
- net BOOT0: now also R1.2, U1.60 (BOOT0), JP4.2 (B); no longer R1.1
- net ENC1_BTN: no longer U1.35 (PB14)
- net ENC2_BTN: now also U1.16 (PA2); no longer U1.34 (PB13)
- net GND: now also D6.1 (K), J1.SH1 (SHIELD), J1.SH2 (SHIELD__1), J1.SH3 (SHIELD__2), J1.SH4 (SHIELD__3), R1.1, R5.2, SW7.S2, J2.1 (Pin_1), J5.3 (Pin_3), J6.1 (Pin_1), J7.2 (Pin_2), SW2.1, SW2.3, SW3.1, SW3.3, SW4.1, SW4.3, SW5.1, SW5.3; no longer R2.2, SW7.S1
- net I2C1_SCL: now also J5.2 (Pin_2); no longer U1.58 (PB6)
- net I2C1_SDA: now also J5.1 (Pin_1); no longer U1.59 (PB7)
- net PUSH_BTN1: now also U1.57 (PB5); no longer U1.27 (PB1)
- net PUSH_BTN2: now also U1.2 (PC13); no longer U1.28 (PB2)
- net PUSH_BTN3: now also U1.3 (PC14); no longer U1.11 (PC3)
- net PUSH_BTN4: now also U1.4 (PC15), U3.12 (6Y); no longer U1.24 (PC4), U3.8 (4Y)
- net RFM_EN: now also U1.24 (PC4), J7.3 (Pin_3); no longer U1.26 (PB0)
- net RFM_G0: now also U1.26 (PB0), J7.9 (Pin_9)
- net RFM_nRST: now also J7.8 (Pin_8)
- net SPI1_MISO: now also J7.5 (Pin_5)
- net SPI1_MOSI: now also J7.6 (Pin_6)
- net SPI1_SCK: now also J7.4 (Pin_4)
- net SPI1_nCS: now also J7.7 (Pin_7)
- net ST7735_DC: now also U1.56 (PB4), J6.6 (Pin_6); no longer U1.16 (PA2)
- net SWCLK: now also J4.3 (Pin_3); no longer J4.4 (Pin_4)
- net TIM2_CH1: now also U4.12 (6Y); no longer U4.2 (1Y)
- net TIM2_CH2: now also U4.10 (5Y); no longer U4.4 (2Y)
- net USART_RX: no longer U1.38 (PC7)
- net USART_TX: no longer U1.37 (PC6)
- net VBUS: no longer C19.2, J3.1 (VBUS), L2.1
- net SW2: now reaches C23.2, R16.1, U3.1 (1A)
- net SW2: now also SW2.2, SW2.4
- net ENC1_SW: now reaches C29.1, R22.2, SW6.S1, U4.5 (3A)
- net ENC1_C: now reaches C28.1, R21.2, SW6.A, U4.3 (2A)
- net ENC1_A: now reaches C27.2, R20.1, SW6.B, U4.1 (1A)
- net OSC_IN: now reaches X1.1
- net OSC_IN: now also C14.2, U1.5 (PH0); no longer U1.3 (PC14)
- net nRST: now reaches C33.2, SW1.1, SW1.3, U1.7 (NRST)
- net nRST: now also J4.4 (Pin_4); no longer J4.3 (Pin_3)
- net REG_IN: now reaches C16.1, D4.1 (K), D5.1 (K), R10.1, U2.1 (VI)
- net SW3: now reaches C24.2, R17.1, U3.3 (2A)
- net SW3: now also SW3.2, SW3.4
- net USB_OTG_FS+: now reaches J1.B6 (DP2)
- net USB_OTG_FS+: now also D2.1 (A1), U1.45 (PA12)
- net USB_OTG_FS-: now reaches J1.B7 (DN2)
- net USB_OTG_FS-: now also D1.1 (A1), U1.44 (PA11)
- net SW4: now reaches C25.2, R19.1, U3.5 (3A)
- net SW4: now also SW4.2, SW4.4
- net ENC2_A: now reaches C30.2, R23.1, U4.13 (6A)
- net ENC2_A: now also SW7.B; no longer SW7.A
- net ENC2_C: now reaches C31.2, R24.1, U4.11 (5A)
- net ENC2_C: now also SW7.A; no longer SW7.B
- net ENC2_SW: now reaches C32.2, R25.1, U4.9 (4A)
- net ENC2_SW: now also SW7.S1; no longer SW7.S2
- net D-: now reaches C20.1, J3.2 (D-), R13.2
- net D+: now reaches C21.1, J3.3 (D+), R12.1
- net SW5: now reaches C26.1, R18.2
- net SW5: now also U3.13 (6A), SW5.2, SW5.4; no longer U3.9 (4A)
- net V_USB: now reaches D4.2 (A), F1.2, Q1.2 (G)
- net at U6.14 (CBUS1): no longer D6.1 (K)
- net at D6.2 (A): now also R2.1
- net at R5.1: now also JP1.1 (A), J6.8 (Pin_8)
- net V_BAT: now reaches D5.2 (A), Q1.1 (D)
- net OSC_OUT: now reaches C13.2
- net OSC_OUT: now also U1.6 (PH1), X1.3; no longer U1.5 (PH0)
- net MCU_LED: now reaches R6.2
- net MCU_LED: now also U1.28 (PB2); no longer U1.51 (PC10)
- net USBD-: now reaches R12.2, U6.9 (USBDM)
- net USBD+: now reaches R13.1, U6.8 (USBDP)
- net ADC_CURRENT_SENSE: no longer names the net of U1.8 (PC0)
- net PA15 renamed SPI3_nCS
- net SPI3_nCS: now also J6.7 (Pin_7)
- net PA8: no longer names the net of U1.41 (PA8)
- net PB3: no longer names the net of U1.55 (PB3)
- net PC11: no longer names the net of U1.52 (PC11)
- net PC12 renamed SPI3_MOSI
- net SPI3_MOSI: now also J6.4 (Pin_4)
- net PC8: no longer names the net of U1.39 (PC8)
- net PC9: no longer names the net of U1.40 (PC9)
- net PD2 renamed ST7735_nRST
- net ST7735_nRST: now also J6.5 (Pin_5)
- net RFM__G0: no longer names the net of U1.10 (PC2)
- net SPI2_MOSI: no longer names the net of U1.36 (PB15)
- net SPI2_NSS: no longer names the net of U1.33 (PB12)
- net SPI2_SCK renamed HB_LED
- net HB_LED: now also R2.2
- removed net TIM3_CH1: U1.56 (PB4), U4.12 (6Y)
- removed net TIM3_CH2: U1.57 (PB5), U4.10 (5Y)
- removed net USB_OTG_FS_DM-: D1.1 (A1), J1.A7 (DN1), U1.44 (PA11)
- removed net USB_OTG_FS_DP+: D2.1 (A1), J1.A6 (DP1), U1.45 (PA12)
- new net: C19.2, J3.1 (VBUS), L2.1
- new net SPI3_SCK: J6.3 (Pin_3), U1.51 (PC10)
- new net TIM4_CH1: U1.58 (PB6), U4.2 (1Y)
- new net TIM4_CH2: U1.59 (PB7), U4.4 (2Y)
- no-connect marks 41 -> 39
Other:
- moved on the sheet: C13, C14, C22, C23, C24, C25, C26, C27, C28, C29, C30, C31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

Commit message: updates
Parts:
- removed J1: USBC, drone_remote:GCT_USB4105-GF-A, symbol UJ20-C-H-G-MSMT-3-P16-TR:UJ20-C-H-G-MSMT-3-P16-TR
- added J3: GSB1C411101DS1HR, pcb_project:AMPHENOL_GSB1C411101DS1HR, symbol GSB1C411101DS1HR:GSB1C411101DS1HR
- C1: renamed from C20; footprint Capacitor_SMD:C_0201_0603Metric -> Capacitor_SMD:C_0402_1005Metric
- C2: renamed from C21; footprint Capacitor_SMD:C_0201_0603Metric -> Capacitor_SMD:C_0402_1005Metric
- D6: footprint Inductor_SMD:L_0201_0603Metric -> LED_SMD:LED_0603_1608Metric
- D7: renamed from D10; footprint Resistor_SMD:R_0201_0603Metric -> LED_SMD:LED_0603_1608Metric
- D8: renamed from D9; footprint LED_SMD:LED_0201_0603Metric -> LED_SMD:LED_0603_1608Metric
- H1, H2, H3, H4: footprint MountingHole:MountingHole_2.2mm_M2 -> MountingHole:MountingHole_2.7mm_M2.5
- J2: renamed from J3; footprint 690-005-299-043_EDA:690-005-299-043_EDA -> pcb_project:CONN5_USB1734035_NP_TEC
- SW1, SW4, SW5: footprint SW4_1825910-B_TEC:SW4_1825910-B_TEC -> pcb_project:SW_1825910-6-4
- SW2: renamed from SW3; footprint SW4_1825910-B_TEC:SW4_1825910-B_TEC -> pcb_project:SW_1825910-6-4
- SW3: renamed from SW2; footprint SW4_1825910-B_TEC:SW4_1825910-B_TEC -> pcb_project:SW_1825910-6-4
- SW6, SW7: footprint Rotary_Encoder:RotaryEncoder_Alps_EC11E-Switch_Vertical_H20mm -> Rotary_Encoder:RotaryEncoder_Bourns_Vertical_PEC12R-3x17F-Sxxxx
- U3: footprint SN74ALVC14PWR:PW14 -> Package_SO:SSOP-16_3.9x4.9mm_P0.635mm
- U4: footprint SN74ALVC14PWR:PW14 -> Package_SO:SSOP-14_5.3x6.2mm_P0.65mm
- X1: footprint ECS-80-10:SMD_ECS-80-10-3M-TR_ECS -> pcb_project:XTAL_ECS-80-10-30B-CWN-TR
- renumbered C3 to C10, C2 to C11, C8 to C12, C9 to C13, C10 to C14, C1 to C15, C14 to C16, C13 to C17, C15 to C18, C16 to C19, C17 to C20, C24 to C21, C25 to C22, C26 to C24, C27 to C25, C28 to C26, C29 to C27, C31 to C28, C32 to C29, C19 to C3, C33 to C4, C22 to C5, C7 to C6, C6 to C7, C5 to C8, C4 to C9, D5 to D4, D4 to D5, J4 to J1, J2 to J4, J6 to J5, J5 to J6, JP4 to JP1, JP1 to JP2, L2 to L1, L1 to L2, R8 to R1, R17 to R10, R10 to R11, R11 to R12, R16 to R13, R19 to R14, R18 to R15, R5 to R16, R26 to R17, R20 to R18, R21 to R19, R12 to R2, R22 to R20, R23 to R21, R24 to R22, R25 to R23, R13 to R3, R7 to R4, R1 to R5, R2 to R6, R6 to R7, R3 to R8, R4 to R9, U6 to U5
Connections:
- net +3.3V: now also R8.1, R9.1; no longer R8.2, R9.2
- net GND: now also R1.1, J3.A1B12 (GND_A), J3.B1A12 (GND_B); no longer R1.2
- net SW2: now also U3.3 (2A); no longer U3.1 (1A)
- net SW3: now also U3.5 (3A); no longer U3.3 (2A)
- net SW4: now also U3.1 (1A); no longer U3.5 (3A)
- net SWCLK: now also R9.2; no longer R9.1
- net SWDIO: now also R8.2; no longer R8.1
- net USB_OTG_FS+: now also J3.A6 (D1+), J3.B6 (D2+)
- net USB_OTG_FS-: now also J3.A7 (D1-), J3.B7 (D2-)
- net VBUS: now also J3.A4B9 (VBUS_A), J3.B4A9 (VBUS_B)
- net at R4.1: now also J3.B5 (CC2)
- new net: J3.A5 (CC1), R1.2
- no-connect marks 39 -> 42
Other:
- moved on the sheet: C18, C19, C20, D1, D2, D3, D4, D5, F1, J4, Q1, R1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

Commit message: finalised first version of pcb, generated manufacturing files, cleaned up file dir
Parts:
- removed JP1: Jumper_2_Bridged, Connector_PinHeader_2.54mm:PinHeader_1x02_P2.54mm_Vertical, symbol Jumper:Jumper_2_Bridged
- added R24: 10k, Resistor_SMD:R_0402_1005Metric, symbol Device:R
- added R25: 10k, Resistor_SMD:R_0805_2012Metric, symbol Device:R_Small
- D1, D2, D3: footprint Diode_SMD:D_0402_1005Metric -> Diode_SMD:D_SOD-323
- J2: footprint pcb_project:CONN5_USB1734035_NP_TEC -> project_library:CONN5_USB1734035_NP_TEC
- J3: footprint pcb_project:AMPHENOL_GSB1C411101DS1HR -> project_library:AMPHENOL_GSB1C411101DS1HR
- SW1, SW2, SW3, SW4, SW5: footprint pcb_project:SW_1825910-6-4 -> project_library:SW_1825910-6-4
- SW6, SW7: footprint Rotary_Encoder:RotaryEncoder_Bourns_Vertical_PEC12R-3x17F-Sxxxx -> Rotary_Encoder:RotaryEncoder_Alps_EC11E-Switch_Vertical_H20mm
- U3: footprint Package_SO:SSOP-16_3.9x4.9mm_P0.635mm -> SN74ALVC14PWR:PW14
- U4: footprint Package_SO:SSOP-14_5.3x6.2mm_P0.65mm -> SN74ALVC14PWR:PW14
- X1: footprint pcb_project:XTAL_ECS-80-10-30B-CWN-TR -> project_library:SMD_ECS-80-10-3M-TR_ECS
Connections:
- net +3.3V: now also R24.2, R25.1
- net BOOT0: now also R25.2
- net RFM_EN: no longer names the net of J7.3 (Pin_3)
- net RFM_EN: now also R24.1; no longer U1.24 (PC4)
- no-connect marks 42 -> 43
Other:
- company: (none) -> Ryan Kelly
- title: (none) -> Drone Remote
- moved on the sheet: C1, C10, C11, C12, C13, C14, C15, C16, C17, C2, C21, C22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

Commit message: some images
Other:
- note added: "Display"
- note added: "Input"
- note added: "MCU"
- note added: "PCB Mounting Holes"
- note added: "Power Input"
- note added: "Radio"
- note added: "USB-B UART"
- title: Drone Remote -> Senser Server
Changed lines of the file:
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@@
 	(paper "A3")
 	(title_block
-		(title "Drone Remote")
-		(date "2025-01-09")
-		(rev "0.1")
+		(title "Senser Server")
+		(date "2025-01-16")
+		(rev "0.2")
 		(company "Ryan Kelly")
 	)
@@
 		)
 	)
+	(text "Display"
+		(exclude_from_sim no)
+		(at 327.914 17.526 0)
+		(effects
+			(font
+				(size 1.27 1.27)
+			)
+		)
+	)
+	(text "USB-B UART"
+		(exclude_from_sim no)
+		(at 135.128 92.202 0)
+		(effects
+			(font
+				(size 1.27 1.27)
+			)
+		)
+	)
+	(text "MCU"
+		(exclude_from_sim no)
+		(at 23.114 161.544 0)
+		(effects
+			(font
+				(size 1.27 1.27)
+			)
+		)
+	)
+	(text "PCB Mounting Holes"
+		(exclude_from_sim no)
+		(at 34.798 97.282 0)
+		(effects
+			(font
+				(size 1.27 1.27)
+			)
+		)
+	)
+	(text "Input"
+		(exclude_from_sim no)
+		(at 249.428 94.742 0)
+		(effects
+			(font
+				(size 1.27 1.27)
+			)
+		)
+	)
+	(text "Power Input"
+		(exclude_from_sim no)
+		(at 34.036 17.018 0)
+		(effects
+			(font
+				(size 1.27 1.27)
+			)
+		)
+	)
+	(text "Radio\n"
+		(exclude_from_sim no)
+		(at 250.444 17.272 0)
+		(effects
+			(font
+				(size 1.27 1.27)
+			)
+		)
+	)
